Commit message: 双臂revolute，其他fixed

File: hello_moveit/moveit/urdf/x1.urdf (robot description, URDF)
Before this commit: robot x1, 58 links, 57 joints
Joints:
- joint left_ankle_pitch_joint: type revolute -> fixed
- joint left_ankle_roll_joint: type revolute -> fixed
- joint left_elbow_pitch_joint: type fixed -> revolute
- joint left_elbow_yaw_joint: type fixed -> revolute
- joint left_hip_pitch_joint: type revolute -> fixed
- joint left_hip_roll_joint: type revolute -> fixed
- joint left_hip_yaw_joint: type revolute -> fixed
- joint left_knee_pitch_joint: type revolute -> fixed
- joint left_shoulder_pitch_joint: type fixed -> revolute
- joint left_shoulder_roll_joint: type fixed -> revolute
- joint left_shoulder_yaw_joint: type fixed -> revolute
- joint left_wrist_pitch_joint: type fixed -> revolute
- joint right_ankle_pitch_joint: type revolute -> fixed
- joint right_ankle_roll_joint: type revolute -> fixed
- joint right_elbow_pitch_joint: type fixed -> revolute
- joint right_elbow_yaw_joint: type fixed -> revolute
- joint right_hip_pitch_joint: type revolute -> fixed
- joint right_hip_roll_joint: type revolute -> fixed
- joint right_hip_yaw_joint: type revolute -> fixed
- joint right_knee_pitch_joint: type revolute -> fixed
- joint right_shoulder_pitch_joint: type fixed -> revolute
- joint right_shoulder_roll_joint: type fixed -> revolute
- joint right_shoulder_yaw_joint: type fixed -> revolute
- joint right_wrist_pitch_joint: type fixed -> revolute
