Commit message: add right_wrist_roll_joint

File: x1_moveit_config/config/x1.ros2_control.xacro (robot description, xacro)
@@ -50,4 +50,11 @@
                 <state_interface name="velocity"/>
             </joint>
+              <joint name="right_wrist_roll_joint">
+                <command_interface name="position"/>
+                <state_interface name="position">
+                  <param name="initial_value">${initial_positions['right_wrist_roll_joint']}</param>
+                </state_interface>
+                <state_interface name="velocity"/>
+            </joint>
         </ros2_control>
     </xacro:macro>

File: x1_moveit_urdf/urdf/x1.urdf (robot description, URDF)
Before this commit: robot x1, 58 links, 57 joints
Links:
- added link left_middle_link
- added link right_middle_link
Joints:
- added joint left_wrist_roll_joint: type revolute, parent left_middle_link, child left_wrist_pitch, origin xyz=0 0 0 rpy=0 0 0, axis 0 1 0, limit lower=-3.14 upper=3.14 effort=0 velocity=0
- added joint right_wrist_roll_joint: type revolute, parent right_middle_link, child right_wrist_pitch, origin xyz=0 0 0 rpy=0 0 0, axis 0 1 0, limit lower=-3.14 upper=3.14 effort=0 velocity=0
- joint left_wrist_pitch_joint: child left_wrist_pitch -> left_middle_link
- joint right_wrist_pitch_joint: child right_wrist_pitch -> right_middle_link
