Commit message: mojia 轨迹录制

File: x1_moveit_urdf/urdf/mojia_old.urdf (robot description, URDF)
Before this commit: robot mojia, 26 links, 25 joints
Links:
- link base_link: geometry visual mesh filename=../meshes2/base_link_simple.STL
- link left_ankle_pitch: geometry visual mesh filename=../meshes2/left_ankle_pitch_simple.STL
- link left_ankle_roll: geometry visual mesh filename=../meshes2/left_ankle_roll_simple.STL
- link left_elbow_pitch: geometry visual mesh filename=../meshes2/left_elbow_pitch_simple.STL
- link left_elbow_yaw: geometry visual mesh filename=../meshes2/left_elbow_yaw_simple.STL
- link left_hip_pitch: geometry visual mesh filename=../meshes2/left_hip_pitch_simple.STL
- link left_hip_roll: geometry visual mesh filename=../meshes2/left_hip_roll_simple.STL
- link left_hip_yaw: geometry visual mesh filename=../meshes2/left_hip_yaw_simple.STL
- link left_knee_pitch: geometry visual mesh filename=../meshes2/left_knee_pitch_simple.STL
- link left_shoulder_pitch: geometry visual mesh filename=../meshes2/left_shoulder_pitch_simple.STL
- link left_shoulder_roll: geometry visual mesh filename=../meshes2/left_shoulder_roll_simple.STL
- link left_shoulder_yaw: geometry visual mesh filename=../meshes2/left_shoulder_yaw_simple.STL
- link lumbar_pitch: geometry visual mesh filename=../meshes2/lumbar_pitch_simple.STL
- link lumbar_roll: geometry visual mesh filename=../meshes2/lumbar_roll_simple.STL
- link lumbar_yaw: geometry visual mesh filename=../meshes2/lumbar_yaw_simple.STL
- link right_ankle_pitch: geometry visual mesh filename=../meshes2/right_ankle_pitch_simple.STL
- link right_ankle_roll: geometry visual mesh filename=../meshes2/right_ankle_roll_simple.STL
- link right_elbow_pitch: geometry visual mesh filename=../meshes2/right_elbow_pitch_simple.STL
- link right_elbow_yaw: geometry visual mesh filename=../meshes2/right_elbow_yaw_simple.STL
- link right_hip_pitch: geometry visual mesh filename=../meshes2/right_hip_pitch_simple.STL
- link right_hip_roll: geometry visual mesh filename=../meshes2/right_hip_roll_simple.STL
- link right_hip_yaw: geometry visual mesh filename=../meshes2/right_hip_yaw_simple.STL
- link right_knee_pitch: geometry visual mesh filename=../meshes2/right_knee_pitch_simple.STL
- link right_shoulder_pitch: geometry visual mesh filename=../meshes2/right_shoulder_pitch_simple.STL
- link right_shoulder_roll: geometry visual mesh filename=../meshes2/right_shoulder_roll_simple.STL
- link right_shoulder_yaw: geometry visual mesh filename=../meshes2/right_shoulder_yaw_simple.STL
