Commit message: x1_moveit_service

File: x1_moveit_urdf/urdf/x1.urdf (robot description, URDF)
Before this commit: robot x1, 58 links, 57 joints
Links:
- link arm_l_wrist_a_ball: geometry visual mesh filename=package://x1_moveit_urdf/meshes/arm_r_wrist_a_ball.STL
- link arm_l_wrist_a_loop: geometry visual mesh filename=package://x1_moveit_urdf/meshes/arm_r_wrist_a_loop.STL
- link arm_l_wrist_b_ball: geometry visual mesh filename=package://x1_moveit_urdf/meshes/arm_r_wrist_b_ball.STL
- link arm_l_wrist_b_loop: geometry visual mesh filename=package://x1_moveit_urdf/meshes/arm_r_wrist_b_loop.STL
- link arm_l_wrist_motor_a_link: geometry visual mesh filename=package://x1_moveit_urdf/meshes/arm_r_wrist_motor_a_link.STL
- link arm_l_wrist_motor_b_link: geometry visual mesh filename=package://x1_moveit_urdf/meshes/arm_r_wrist_motor_b_link.STL
- link arm_r_wrist_a_ball: geometry visual mesh filename=package://x1_moveit_urdf/meshes/arm_r_wrist_a_ball.STL
- link arm_r_wrist_a_loop: geometry visual mesh filename=package://x1_moveit_urdf/meshes/arm_r_wrist_a_loop.STL
- link arm_r_wrist_b_ball: geometry visual mesh filename=package://x1_moveit_urdf/meshes/arm_r_wrist_b_ball.STL
- link arm_r_wrist_b_loop: geometry visual mesh filename=package://x1_moveit_urdf/meshes/arm_r_wrist_b_loop.STL
- link arm_r_wrist_motor_a_link: geometry visual mesh filename=package://x1_moveit_urdf/meshes/arm_r_wrist_motor_a_link.STL
- link arm_r_wrist_motor_b_link: geometry visual mesh filename=package://x1_moveit_urdf/meshes/arm_r_wrist_motor_b_link.STL
- link base_link: geometry collision mesh filename=package://x1_moveit_urdf/meshes/base_link_simple.STL; visual mesh filename=package://x1_moveit_urdf/meshes/base_link_simple.STL
- link left_ankle_pitch: geometry visual mesh filename=package://x1_moveit_urdf/meshes/left_ankle_pitch.STL
- link left_ankle_roll: geometry collision mesh filename=package://x1_moveit_urdf/meshes/left_ankle_roll.STL; visual mesh filename=package://x1_moveit_urdf/meshes/left_ankle_roll.STL
- link left_elbow_pitch: geometry visual mesh filename=package://x1_moveit_urdf/meshes/left_elbow_pitch.STL
- link left_elbow_yaw: geometry visual mesh filename=package://x1_moveit_urdf/meshes/left_elbow_yaw.STL
- link left_hip_pitch: geometry visual mesh filename=package://x1_moveit_urdf/meshes/left_hip_pitch.STL
- link left_hip_roll: geometry visual mesh filename=package://x1_moveit_urdf/meshes/left_hip_roll.STL
- link left_hip_yaw: geometry visual mesh filename=package://x1_moveit_urdf/meshes/left_hip_yaw.STL
- link left_knee_pitch: geometry visual mesh filename=package://x1_moveit_urdf/meshes/left_knee_pitch.STL
- link left_shoulder_pitch: geometry visual mesh filename=package://x1_moveit_urdf/meshes/left_shoulder_pitch.STL
- link left_shoulder_roll: geometry visual mesh filename=package://x1_moveit_urdf/meshes/left_shoulder_roll.STL
- link left_shoulder_yaw: geometry visual mesh filename=package://x1_moveit_urdf/meshes/left_shoulder_yaw.STL
- link left_wrist_pitch: geometry visual mesh filename=package://x1_moveit_urdf/meshes/left_wrist_pitch.STL
- link leg_l_toe_a_ball: geometry visual mesh filename=package://x1_moveit_urdf/meshes/leg_l_toe_a_ball.STL
- link leg_l_toe_a_link: geometry visual mesh filename=package://x1_moveit_urdf/meshes/leg_l_toe_a_link.STL
- link leg_l_toe_a_loop: geometry visual mesh filename=package://x1_moveit_urdf/meshes/leg_l_toe_a_loop.STL
- link leg_l_toe_b_ball: geometry visual mesh filename=package://x1_moveit_urdf/meshes/leg_l_toe_b_ball.STL
- link leg_l_toe_b_link: geometry visual mesh filename=package://x1_moveit_urdf/meshes/leg_l_toe_b_link.STL
- link leg_l_toe_b_loop: geometry visual mesh filename=package://x1_moveit_urdf/meshes/leg_l_toe_b_loop.STL
- link leg_r_toe_a_ball: geometry visual mesh filename=package://x1_moveit_urdf/meshes/leg_r_toe_a_ball.STL
- link leg_r_toe_a_link: geometry visual mesh filename=package://x1_moveit_urdf/meshes/leg_r_toe_a_link.STL
- link leg_r_toe_a_loop: geometry visual mesh filename=package://x1_moveit_urdf/meshes/leg_r_toe_a_loop.STL
- link leg_r_toe_b_ball: geometry visual mesh filename=package://x1_moveit_urdf/meshes/leg_r_toe_b_ball.STL
- link leg_r_toe_b_link: geometry visual mesh filename=package://x1_moveit_urdf/meshes/leg_r_toe_b_link.STL
- link leg_r_toe_b_loop: geometry visual mesh filename=package://x1_moveit_urdf/meshes/leg_r_toe_b_loop.STL
- link lumber_pitch: geometry visual mesh filename=package://x1_moveit_urdf/meshes/lumber_pitch.STL
- link lumber_roll: geometry visual mesh filename=package://x1_moveit_urdf/meshes/lumber_roll.STL
- link lumber_yaw: geometry visual mesh filename=package://x1_moveit_urdf/meshes/lumber_yaw.STL
- link right_ankle_pitch: geometry visual mesh filename=package://x1_moveit_urdf/meshes/right_ankle_pitch.STL
- link right_ankle_roll: geometry collision mesh filename=package://x1_moveit_urdf/meshes/right_ankle_roll.STL; visual mesh filename=package://x1_moveit_urdf/meshes/right_ankle_roll.STL
- link right_elbow_pitch: geometry visual mesh filename=package://x1_moveit_urdf/meshes/right_elbow_pitch.STL
- link right_elbow_yaw: geometry visual mesh filename=package://x1_moveit_urdf/meshes/right_elbow_yaw.STL
- link right_hip_pitch: geometry visual mesh filename=package://x1_moveit_urdf/meshes/right_hip_pitch.STL
- link right_hip_roll: geometry visual mesh filename=package://x1_moveit_urdf/meshes/right_hip_roll.STL
- link right_hip_yaw: geometry visual mesh filename=package://x1_moveit_urdf/meshes/right_hip_yaw.STL
- link right_knee_pitch: geometry visual mesh filename=package://x1_moveit_urdf/meshes/right_knee_pitch.STL
- link right_shoulder_pitch: geometry visual mesh filename=package://x1_moveit_urdf/meshes/right_shoulder_pitch.STL
- link right_shoulder_roll: geometry visual mesh filename=package://x1_moveit_urdf/meshes/right_shoulder_roll.STL
- link right_shoulder_yaw: geometry visual mesh filename=package://x1_moveit_urdf/meshes/right_shoulder_yaw.STL
- link right_wrist_pitch: geometry visual mesh filename=package://x1_moveit_urdf/meshes/right_wrist_pitch.STL
- link waist_motor_a_ball: geometry visual mesh filename=package://x1_moveit_urdf/meshes/waist_motor_a_ball.STL
- link waist_motor_a_link: geometry visual mesh filename=package://x1_moveit_urdf/meshes/waist_motor_a_link.STL
- link waist_motor_a_loop: geometry visual mesh filename=package://x1_moveit_urdf/meshes/waist_motor_a_loop.STL
- link waist_motor_b_ball: geometry visual mesh filename=package://x1_moveit_urdf/meshes/waist_motor_b_ball.STL
- link waist_motor_b_link: geometry visual mesh filename=package://x1_moveit_urdf/meshes/waist_motor_b_link.STL
- link waist_motor_b_loop: geometry visual mesh filename=package://x1_moveit_urdf/meshes/waist_motor_b_loop.STL

Commit message: remove config

File: x1_moveit_urdf/urdf/x1.urdf (robot description, URDF)
Before this commit: robot x1, 58 links, 57 joints
Links:
- added link dummy_base; collision box size=0.001 0.001 0.001; visual box size=0.001 0.001 0.001
- link lumber_pitch: geometry collision mesh filename=package://x1_moveit_urdf/meshes/lumber_pitch.STL; visual mesh filename=package://x1_moveit_urdf/meshes/lumber_pitch.STL
- link lumber_roll: geometry collision mesh filename=package://x1_moveit_urdf/meshes/lumber_roll.STL; visual mesh filename=package://x1_moveit_urdf/meshes/lumber_roll.STL
- link lumber_yaw: geometry collision mesh filename=package://x1_moveit_urdf/meshes/lumber_yaw.STL; visual mesh filename=package://x1_moveit_urdf/meshes/lumber_yaw.STL
Joints:
- added joint dummy_to_base: type fixed, parent dummy_base, child base_link, origin xyz=0 0 0 rpy=0 0 0

Commit message: joycon发布pose

File: x1_moveit_urdf/urdf/x1.urdf (robot description, URDF)
Before this commit: robot x1, 59 links, 58 joints
Links:
- removed link dummy_base
Joints:
- removed joint dummy_to_base

Commit message: 添加shoudler碰撞

File: x1_moveit_urdf/urdf/x1.urdf (robot description, URDF)
Before this commit: robot x1, 60 links, 59 joints
Links:
- link right_elbow_pitch: geometry collision mesh filename=package://x1_moveit_urdf/meshes/right_elbow_pitch.STL; visual mesh filename=package://x1_moveit_urdf/meshes/right_elbow_pitch.STL
- link right_shoulder_roll: geometry collision mesh filename=package://x1_moveit_urdf/meshes/right_shoulder_roll.STL; visual mesh filename=package://x1_moveit_urdf/meshes/right_shoulder_roll.STL

Commit message: right关节limit，日志

File: x1_moveit_urdf/urdf/x1.urdf (robot description, URDF)
Before this commit: robot x1, 60 links, 59 joints
Joints:
- joint right_elbow_pitch_joint: limit lower=-3.14 upper=3.14 effort=0 velocity=0 -> lower=-1.57 upper=1.57 effort=0 velocity=0
- joint right_elbow_yaw_joint: limit lower=-3.14 upper=3.14 effort=0 velocity=0 -> lower=-1.57 upper=1.57 effort=0 velocity=0
- joint right_shoulder_pitch_joint: limit lower=-3.14 upper=3.14 effort=0 velocity=0 -> lower=-1.57 upper=1.57 effort=0 velocity=0
- joint right_shoulder_roll_joint: limit lower=-3.14 upper=3.14 effort=0 velocity=0 -> lower=-1.57 upper=1.57 effort=0 velocity=0
- joint right_shoulder_yaw_joint: limit lower=-3.14 upper=3.14 effort=0 velocity=0 -> lower=-1.57 upper=1.57 effort=0 velocity=0
- joint right_wrist_pitch_joint: limit lower=-3.14 upper=3.14 effort=0 velocity=0 -> lower=-1.57 upper=1.57 effort=0 velocity=0
- joint right_wrist_roll_joint: limit lower=-3.14 upper=3.14 effort=0 velocity=0 -> lower=-1.57 upper=1.57 effort=0 velocity=0

Commit message: 加方块爪子

File: x1_moveit_urdf/urdf/x1.urdf (robot description, URDF)
Before this commit: robot x1, 60 links, 59 joints
Links:
- added link OmniPicker_right; collision box size=0.1 0.1 0.1; visual box size=0.1 0.1 0.1
Joints:
- added joint joint_OmniPicker_right_attachment: type fixed, parent right_wrist_pitch, child OmniPicker_right, origin xyz=0 0 0 rpy=0 0 0

Commit message: moveit 添加深度相机避障： urdf确定位置，sensors_3d.yaml将点云转成八叉树

File: x1_moveit_urdf/urdf/x1.urdf (robot description, URDF)
Before this commit: robot x1, 61 links, 60 joints
Links:
- added link camera_depth_optical_frame
Joints:
- added joint camera_joint: type fixed, parent base_link, child camera_depth_optical_frame, origin xyz=0 0 0.5 rpy=-1.57 0 -1.57
